Commit message: Imported upstream version '0.7.3' of 'upstream'

File: jackal_description/urdf/accessories.urdf.xacro (robot description, xacro)
@@ -13,25 +13,75 @@
   <!-- This optional plate mounts both the upgraded GPS and the Velodyne 3D LIDAR. -->
   <xacro:include filename="$(find jackal_description)/urdf/accessories/bridge_plate.urdf.xacro" />
-  <!-- If enabled, generate the LASER payload (by default, a SICK LMS111). -->
+  <xacro:include filename="$(find jackal_description)/urdf/accessories/sick_lms1xx_mount.urdf.xacro" />
+  <xacro:include filename="$(find jackal_description)/urdf/accessories/hokuyo_ust10.urdf.xacro" />
+  <xacro:include filename="$(find jackal_description)/urdf/accessories/vlp16_mount.urdf.xacro" />
+  <!--
+    Add primary/secondary 2D lidar sensors.  By default these are SICK LMS1xx but can be changed with the
+    JACKAL_LASER_MODEL and JACKAL_LASER_SECONDARY_MODEL environment variables. Valid model designations are:
+    - lms1xx (default) :: SICK LMS1xx
+    - ust10            :: Hokuyo UST10
+  -->
   <xacro:if value="$(optenv JACKAL_LASER 0)">
-    <xacro:if value="$(optenv JACKAL_LASER_HOKUYO 0)">
+    <xacro:property name="lidar_model" value="$(optenv JACKAL_LASER_MODEL lms1xx)" />
+    <xacro:if value="${lidar_model == 'lms1xx'}">
+      <xacro:include filename="$(find jackal_description)/urdf/accessories/sick_lms1xx_mount.urdf.xacro" />
+      <xacro:sick_lms1xx_mount prefix="$(optenv JACKAL_LASER_MOUNT front)"
+           parent_link="$(optenv JACKAL_LASER_MOUNT front)_mount"
+           topic="$(optenv JACKAL_LASER_TOPIC front/scan)">
+        <origin xyz="$(optenv JACKAL_LASER_OFFSET 0 0 0)"
+                   rpy="$(optenv JACKAL_LASER_RPY 0 0 0)" />
+      </xacro:sick_lms1xx_mount>
+    </xacro:if>
+    <xacro:if value="${lidar_model == 'ust10'}">
       <xacro:include filename="$(find jackal_description)/urdf/accessories/hokuyo_ust10.urdf.xacro" />
-      <hokuyo_ust10_mount prefix="$(optenv JACKAL_LASER_MOUNT front)"
-                          parent_link="$(optenv JACKAL_LASER_MOUNT front)_mount"
-                          topic="$(optenv JACKAL_LASER_TOPIC front/scan)" />
+      <xacro:hokuyo_ust10_mount prefix="$(optenv JACKAL_LASER_MOUNT front)"
+          parent_link="$(optenv JACKAL_LASER_MOUNT front)_mount"
+          topic="$(optenv JACKAL_LASER_TOPIC front/scan)">
+        <origin xyz="$(optenv JACKAL_LASER_OFFSET 0 0 0)"
+                rpy="$(optenv JACKAL_LASER_RPY 0 0 0)" />
+      </xacro:hokuyo_ust10_mount>
     </xacro:if>
-    <xacro:unless value="$(optenv JACKAL_LASER_HOKUYO 0)">
-      <xacro:include filename="$(find jackal_description)/urdf/accessories/sick_lms1xx_mount.urdf.xacro" />
-      <sick_lms1xx_mount prefix="$(optenv JACKAL_LASER_MOUNT front)"
-                         parent_link="$(optenv JACKAL_LASER_MOUNT front)_mount"
-                         topic="$(optenv JACKAL_LASER_TOPIC front/scan)"/>
-    </xacro:unless>
+  </xacro:if>
+  <xacro:if value="$(optenv JACKAL_LASER_SECONDARY 0)">
+    <xacro:property name="lidar2_model" value="$(optenv JACKAL_LASER_SECONDARY_MODEL lms1xx)" />
+    <xacro:if value="${lidar2_model == 'lms1xx'}">
+      <xacro:sick_lms1xx_mount prefix="$(optenv JACKAL_LASER_SECONDARY_MOUNT rear)"
+           parent_link="$(optenv JACKAL_LASER_SECONDARY_MOUNT rear)_mount"
+           topic="$(optenv JACKAL_LASER_SECONDARY_TOPIC rear/scan)">
+         <origin xyz="$(optenv JACKAL_LASER_SECONDARY_OFFSET 0 0 0)"
+                 rpy="$(optenv JACKAL_LASER_SECONDARY_RPY 0 0 3.14159)" />
+       </xacro:sick_lms1xx_mount>
+    </xacro:if>
+    <xacro:if value="${lidar2_model == 'ust10'}">
+      <xacro:hokuyo_ust10_mount prefix="$(optenv JACKAL_LASER_SECONDARY_MOUNT rear)"
+          parent_link="$(optenv JACKAL_LASER_SECONDARY_MOUNT rear)_mount"
+          topic="$(optenv JACKAL_LASER_SECONDARY_TOPIC rear/scan)">
+        <origin xyz="$(optenv JACKAL_LASER_SECONDARY_OFFSET 0 0 0)"
+                rpy="$(optenv JACKAL_LASER_SECONDARY_RPY 0 0 3.14159)" />
+      </xacro:hokuyo_ust10_mount>
+    </xacro:if>
+  </xacro:if>
+  <!--
+    Add a 3D lidar sensor.  By default this is a Velodyne VLP16 but can be changed with the
+    JACKAL_LASER_3D_MODEL environment variable. Valid model designations are:
+    - vlp16 (default)  :: Velodyne VLP16
+  -->
+  <xacro:if value="$(optenv JACKAL_LASER_3D 0)">
+    <xacro:property name="lidar_3d_model" value="$(optenv JACKAL_LASER_3D_MODEL vlp16)" />
+    <xacro:if value="${lidar_3d_model == 'vlp16'}">
+      <xacro:vlp16_mount
+          parent_link="$(optenv JACKAL_LASER_3D_MOUNT mid)_mount"
+          prefix="$(optenv JACKAL_LASER_3D_MOUNT mid)"
+          topic="$(optenv JACKAL_LASER_3D_TOPIC mid/points)">
+        <origin xyz="$(optenv JACKAL_LASER_3D_OFFSET 0 0 0)" rpy="$(optenv JACKAL_LASER_3D_RPY 0 0 0)" />
+      </xacro:vlp16_mount>
+    </xacro:if>
   </xacro:if>
   <!-- If enabled, generate the upgraded Navsat payload (a Novatel Smart6). -->
   <xacro:if value="$(optenv JACKAL_NAVSAT 0)">
     <xacro:include filename="$(find jackal_description)/urdf/accessories/novatel_smart6.urdf.xacro" />
-    <bridge_plate mount="$(optenv JACKAL_NAVSAT_MOUNT rear)"
+    <xacro:bridge_plate mount="$(optenv JACKAL_NAVSAT_MOUNT rear)"
                   height="$(optenv JACKAL_NAVSAT_HEIGHT 0.1)" />
-    <novatel_smart6 prefix="$(optenv JACKAL_NAVSAT_MOUNT rear)"/>
+    <xacro:novatel_smart6 prefix="$(optenv JACKAL_NAVSAT_MOUNT rear)"/>
     <joint name="$(optenv JACKAL_NAVSAT_MOUNT rear)_navsat_joint" type="fixed">
       <origin xyz="0 0 0" rpy="0 0 0" />
@@ -41,9 +91,9 @@
   </xacro:if>
   <!-- Common camera mounts and accessory URDFs. -->
-  <!-- <xacro:include filename="$(find jackal_description)/urdf/accessories/camera_mount.urdf.xacro" /> -->
-  <!-- <xacro:include filename="$(find pointgrey_camera_description)/urdf/pointgrey_flea3.urdf.xacro" /> -->
+  <xacro:include filename="$(find jackal_description)/urdf/accessories/camera_mount.urdf.xacro" />
+  <xacro:include filename="$(find pointgrey_camera_description)/urdf/pointgrey_flea3.urdf.xacro" />
   <!-- If enabled, generate the flea3 camera payload with a tilt of 30 degrees. -->
-  <!-- <xacro:if value="$(optenv JACKAL_FLEA3 0)">
-    <camera_mount prefix="$(optenv JACKAL_FLEA3_MOUNT front)"
+  <xacro:if value="$(optenv JACKAL_FLEA3 0)">
+    <xacro:camera_mount prefix="$(optenv JACKAL_FLEA3_MOUNT front)"
                        tilt="$(optenv JACKAL_FLEA3_TILT 0.5236)"/>
     <joint name="$(optenv JACKAL_FLEA3_MOUNT front)_camera_mount_joint" type="fixed">
@@ -53,5 +103,5 @@
       <child link="$(optenv JACKAL_FLEA3_MOUNT front)_camera_mount" />
     </joint>
-    <pointgrey_flea3 frame="$(optenv JACKAL_FLEA3_MOUNT front)_camera" name="$(optenv JACKAL_FLEA3_NAME front)"
+    <xacro:pointgrey_flea3 frame="$(optenv JACKAL_FLEA3_MOUNT front)_camera" name="$(optenv JACKAL_FLEA3_NAME front)"
       camera_x="0.0754" camera_y="0.029" camera_z="0.029"
       camera_mass="0.085" hfov="1.0471975512" fps="60" width="640" height="512"/>
@@ -61,10 +111,10 @@
       <child link="$(optenv JACKAL_FLEA3_MOUNT front)_camera" />
     </joint>
-  </xacro:if> -->
-  <!-- <xacro:include filename="$(find jackal_description)/urdf/accessories/stereo_camera_mount.urdf.xacro" /> -->
+  </xacro:if>
+  <xacro:include filename="$(find jackal_description)/urdf/accessories/stereo_camera_mount.urdf.xacro" />
   <!-- If enabled, generates a pair of flea3 cameras for stereo vision with a tilt of 30 degrees. -->
   <!-- Disabled temporarily due to metapackage issue. -->
-  <!-- <xacro:if value="$(optenv JACKAL_STEREO_FLEA3 0)">
-    <stereo_camera_mount prefix="$(optenv JACKAL_FLEA3_MOUNT front)"
+  <xacro:if value="$(optenv JACKAL_STEREO_FLEA3 0)">
+    <xacro:stereo_camera_mount prefix="$(optenv JACKAL_FLEA3_MOUNT front)"
                        tilt="$(optenv JACKAL_FLEA3_TILT 0.5236)"/>
     <joint name="$(optenv JACKAL_FLEA3_MOUNT front)_stereo_camera_mount_joint" type="fixed">
@@ -74,5 +124,5 @@
       <child link="$(optenv JACKAL_FLEA3_MOUNT front)_stereo_camera_mount" />
     </joint>
-    <pointgrey_flea3 frame="$(optenv JACKAL_FLEA3_MOUNT front)_left_camera" name="$(optenv JACKAL_FLEA3_LEFT_NAME front/left)"
+    <xacro:pointgrey_flea3 frame="$(optenv JACKAL_FLEA3_MOUNT front)_left_camera" name="$(optenv JACKAL_FLEA3_LEFT_NAME front/left)"
       camera_x="0.0754" camera_y="0.029" camera_z="0.029"
       camera_mass="0.085" hfov="1.0471975512" fps="60" width="640" height="512"/>
@@ -82,5 +132,5 @@
       <child link="$(optenv JACKAL_FLEA3_MOUNT front)_left_camera" />
     </joint>
-    <pointgrey_flea3 frame="$(optenv JACKAL_FLEA3_MOUNT front)_right_camera" name="$(optenv JACKAL_FLEA3_RIGHT_NAME front/right)"
+    <xacro:pointgrey_flea3 frame="$(optenv JACKAL_FLEA3_MOUNT front)_right_camera" name="$(optenv JACKAL_FLEA3_RIGHT_NAME front/right)"
       camera_x="0.0754" camera_y="0.029" camera_z="0.029"
       camera_mass="0.085" hfov="1.0471975512" fps="60" width="640" height="512"/>
@@ -90,11 +140,11 @@
       <child link="$(optenv JACKAL_FLEA3_MOUNT front)_right_camera" />
     </joint>
-  </xacro:if> -->
+  </xacro:if>
   <!-- If enabled, generate the bumblebee2 camera payload with a tilt of 0 degrees. -->
-  <!-- <xacro:include filename="$(find pointgrey_camera_description)/urdf/pointgrey_bumblebee2.urdf.xacro" /> -->
+  <xacro:include filename="$(find pointgrey_camera_description)/urdf/pointgrey_bumblebee2.urdf.xacro" />
   <!-- If enabled, generate the bumblebee2 camera payload with a tilt of 0 degrees. -->
   <!-- Disabled temporarily due to metapackage issue. -->
-  <!-- <xacro:if value="$(optenv JACKAL_BB2 0)">
-    <camera_mount prefix="$(optenv JACKAL_BB2_MOUNT front)"
+  <xacro:if value="$(optenv JACKAL_BB2 0)">
+    <xacro:camera_mount prefix="$(optenv JACKAL_BB2_MOUNT front)"
                         tilt="$(optenv JACKAL_BB2_TILT 0)"/>
     <joint name="$(optenv JACKAL_BB2_MOUNT front)_camera_mount_joint" type="fixed">
@@ -104,5 +154,5 @@
       <child link="$(optenv JACKAL_BB2_MOUNT front)_camera_mount" />
     </joint>
-    <BB2-08S2C-38 frame="$(optenv JACKAL_BB2_MOUNT front)_camera" name="$(optenv JACKAL_BB2_NAME front)" />
+    <xacro:BB2-08S2C-38 frame="$(optenv JACKAL_BB2_MOUNT front)_camera" name="$(optenv JACKAL_BB2_NAME front)" />
     <joint name="$(optenv JACKAL_BB2_MOUNT front)_camera_bracket_joint" type="fixed">
       <origin xyz="0.007 0 0.02450" rpy="0 0 0" />
@@ -110,9 +160,9 @@
       <child link="$(optenv JACKAL_BB2_MOUNT front)_camera" />
     </joint>
-  </xacro:if> -->
+  </xacro:if>
   <xacro:if value="$(optenv JACKAL_FRONT_ACCESSORY_FENDER 0)">
     <xacro:include filename="$(find jackal_description)/urdf/accessories/hokuyo_ust10.urdf.xacro" />
     <xacro:if value="$(optenv JACKAL_FRONT_FENDER_UST10 0)">
-      <hokuyo_ust10_mount
+      <xacro:hokuyo_ust10_mount
         prefix="front"
         parent_link="front_fender_accessory_link"
@@ -122,5 +172,5 @@
   <xacro:if value="$(optenv JACKAL_REAR_ACCESSORY_FENDER 0)">
     <xacro:if value="$(optenv JACKAL_REAR_FENDER_UST10 0)">
-      <hokuyo_ust10_mount
+      <xacro:hokuyo_ust10_mount
         prefix="rear"
         parent_link="rear_fender_accessory_link"

File: jackal_description/urdf/accessories/hokuyo_ust10.urdf.xacro (robot description, xacro)
@@ -1,5 +1,5 @@
 <?xml version="1.0"?>
 <robot xmlns:xacro="http://ros.org/wiki/xacro">
-  <xacro:macro name="hokuyo_ust10_mount" params="prefix topic parent_link">
+  <xacro:macro name="hokuyo_ust10_mount" params="prefix topic parent_link *origin">
     <xacro:macro name="hokuyo_ust10" params="frame:=laser topic:=scan sample_size:=720 update_rate:=50
                min_angle:=-2.35619 max_angle:=2.35619 min_range:=0.1 max_range:=30.0 robot_namespace:=/">
@@ -47,8 +47,7 @@
       </gazebo>
     </xacro:macro>
-    <hokuyo_ust10 frame="${prefix}_laser" topic="${topic}"/>
+    <xacro:hokuyo_ust10 frame="${prefix}_laser" topic="${topic}"/>
     <joint name="${prefix}_laser_mount_joint" type="fixed">
-      <origin xyz="$(optenv JACKAL_LASER_OFFSET 0 0 0)"
-              rpy="$(optenv JACKAL_LASER_RPY 0 0 0)" />
+      <xacro:insert_block name="origin" />
       <parent link="${parent_link}" />
       <child link="${prefix}_laser_mount" />

File: jackal_description/urdf/accessories/sick_lms1xx_mount.urdf.xacro (robot description, xacro)
@@ -27,9 +27,8 @@
 <robot xmlns:xacro="http://www.ros.org/wiki/xacro">
   <xacro:include filename="$(find lms1xx)/urdf/sick_lms1xx.urdf.xacro" />
-  <xacro:macro name="sick_lms1xx_mount" params="prefix topic parent_link">
-    <sick_lms1xx frame="${prefix}_laser" topic="${topic}" />
+  <xacro:macro name="sick_lms1xx_mount" params="prefix topic parent_link *origin">
+    <xacro:sick_lms1xx frame="${prefix}_laser" topic="${topic}" />
     <joint name="${prefix}_laser_mount_joint" type="fixed">
-      <origin xyz="$(optenv JACKAL_LASER_OFFSET 0 0 0)"
-              rpy="$(optenv JACKAL_LASER_RPY 0 0 0)" />
+      <xacro:insert_block name="origin" />
       <parent link="${parent_link}" />
       <child link="${prefix}_laser_mount" />

Commit message: Imported upstream version '0.7.6' of 'upstream'

File: jackal_description/urdf/accessories.urdf.xacro (robot description, xacro)
@@ -80,8 +80,15 @@
   <!-- If enabled, generate the upgraded Navsat payload (a Novatel Smart6). -->
   <xacro:if value="$(optenv JACKAL_NAVSAT 0)">
-    <xacro:include filename="$(find jackal_description)/urdf/accessories/novatel_smart6.urdf.xacro" />
+    <xacro:property name="navsat_model" value="$(optenv JACKAL_NAVSAT_MODEL smart6)" />
+    <xacro:if value="${navsat_model == 'smart6'}">
+      <xacro:include filename="$(find jackal_description)/urdf/accessories/novatel_smart6.urdf.xacro" />
+      <xacro:novatel_smart6 prefix="$(optenv JACKAL_NAVSAT_MOUNT rear)"/>
+    </xacro:if>
+    <xacro:if value="${navsat_model == 'smart7'}">
+      <xacro:include filename="$(find jackal_description)/urdf/accessories/novatel_smart7.urdf.xacro" />
+      <xacro:novatel_smart7 prefix="$(optenv JACKAL_NAVSAT_MOUNT rear)"/>
+    </xacro:if>
     <xacro:bridge_plate mount="$(optenv JACKAL_NAVSAT_MOUNT rear)"
                   height="$(optenv JACKAL_NAVSAT_HEIGHT 0.1)" />
-    <xacro:novatel_smart6 prefix="$(optenv JACKAL_NAVSAT_MOUNT rear)"/>
     <joint name="$(optenv JACKAL_NAVSAT_MOUNT rear)_navsat_joint" type="fixed">
       <origin xyz="0 0 0" rpy="0 0 0" />
@@ -167,4 +174,6 @@
         prefix="front"
         parent_link="front_fender_accessory_link"
+        min_angle="${-pi/2}"
+        max_angle="${pi/2}"
         topic="$(optenv JACKAL_FRONT_LASER_TOPIC front/scan)">
         <origin xyz="0 0 0" rpy="0 0 0" />
@@ -177,4 +186,6 @@
         prefix="rear"
         parent_link="rear_fender_accessory_link"
+        min_angle="${-pi/2}"
+        max_angle="${pi/2}"
         topic="$(optenv JACKAL_REAR_LASER_TOPIC rear/scan)">
         <origin xyz="0 0 0" rpy="0 0 0" />

File: jackal_description/urdf/jackal.urdf.xacro (robot description, xacro)
@@ -203,4 +203,16 @@
     <origin xyz="-0.180 0.126 0.1815" />
   </joint>
+  <!--
+    Optionally add a GX5 IMU
+  -->
+  <xacro:if value="$(optenv JACKAL_GX5_IMU 0)">
+    <link name="gx5_link" />
+    <joint name="gx5_joint" type="fixed">
+      <parent link="base_link" />
+      <child link="gx5_link" />
+      <!-- TODO This offset & rotation may not be final, but it's good enough for now.  May update, pending RSCI-10 -->
+      <origin xyz="$(optenv JACKAL_GX5_IMU_OFFSET -0.139 0.096 0.100)" rpy="$(optenv JACKAL_GX5_IMU_RPY ${PI} 0 -${PI/2})" />
+    </joint>
+  </xacro:if>
   <link name="mid_mount"></link>
   <joint name="mid_mount_joint" type="fixed">
@@ -229,3 +241,5 @@
   <!-- Optional custom includes. -->
   <xacro:include filename="$(optenv JACKAL_URDF_EXTRAS empty.urdf)" />
+  <!-- Optional for Clearpath internal softwares -->
+  <xacro:include filename="$(optenv CPR_URDF_EXTRAS empty.urdf)" />
 </robot>

Commit message: Imported upstream version '0.8.0' of 'upstream'

File: jackal_description/urdf/accessories.urdf.xacro (robot description, xacro)
@@ -16,5 +16,4 @@
   <xacro:include filename="$(find jackal_description)/urdf/accessories/hokuyo_ust10.urdf.xacro" />
   <xacro:include filename="$(find jackal_description)/urdf/accessories/vlp16_mount.urdf.xacro" />
-  <xacro:include filename="$(find jackal_description)/urdf/accessories/hdl32_mount.urdf.xacro" />
   <!--
     Add primary/secondary 2D lidar sensors.  By default these are SICK LMS1xx but can be changed with the
@@ -67,5 +66,4 @@
     JACKAL_LASER_3D_MODEL environment variable. Valid model designations are:
     - vlp16 (default)  :: Velodyne VLP16
-    - vlp32e           :: Velodyne HDL-32E
   -->
   <xacro:if value="$(optenv JACKAL_LASER_3D 0)">
@@ -75,32 +73,15 @@
           parent_link="$(optenv JACKAL_LASER_3D_MOUNT mid)_mount"
           prefix="$(optenv JACKAL_LASER_3D_MOUNT mid)"
-          topic="$(optenv JACKAL_LASER_3D_TOPIC mid/points)"
-          tower="$(optenv JACKAL_LASER_3D_TOWER 1)">
+          topic="$(optenv JACKAL_LASER_3D_TOPIC mid/points)">
         <origin xyz="$(optenv JACKAL_LASER_3D_OFFSET 0 0 0)" rpy="$(optenv JACKAL_LASER_3D_RPY 0 0 0)" />
       </xacro:vlp16_mount>
     </xacro:if>
-    <xacro:if value="${lidar_3d_model == 'hdl32e'}">
-      <xacro:hdl32e_mount
-          parent_link="$(optenv JACKAL_LASER_3D_MOUNT mid)_mount"
-          prefix="$(optenv JACKAL_LASER_3D_MOUNT mid)"
-          topic="$(optenv JACKAL_LASER_3D_TOPIC mid/points)"
-          tower="$(optenv JACKAL_LASER_3D_TOWER 1)">
-        <origin xyz="$(optenv JACKAL_LASER_3D_OFFSET 0 0 0)" rpy="$(optenv JACKAL_LASER_3D_RPY 0 0 0)" />
-      </xacro:hdl32e_mount>
-    </xacro:if>
   </xacro:if>
   <!-- If enabled, generate the upgraded Navsat payload (a Novatel Smart6). -->
   <xacro:if value="$(optenv JACKAL_NAVSAT 0)">
-    <xacro:property name="navsat_model" value="$(optenv JACKAL_NAVSAT_MODEL smart6)" />
-    <xacro:if value="${navsat_model == 'smart6'}">
-      <xacro:include filename="$(find jackal_description)/urdf/accessories/novatel_smart6.urdf.xacro" />
-      <xacro:novatel_smart6 prefix="$(optenv JACKAL_NAVSAT_MOUNT rear)"/>
-    </xacro:if>
-    <xacro:if value="${navsat_model == 'smart7'}">
-      <xacro:include filename="$(find jackal_description)/urdf/accessories/novatel_smart7.urdf.xacro" />
-      <xacro:novatel_smart7 prefix="$(optenv JACKAL_NAVSAT_MOUNT rear)"/>
-    </xacro:if>
+    <xacro:include filename="$(find jackal_description)/urdf/accessories/novatel_smart6.urdf.xacro" />
     <xacro:bridge_plate mount="$(optenv JACKAL_NAVSAT_MOUNT rear)"
                   height="$(optenv JACKAL_NAVSAT_HEIGHT 0.1)" />
+    <xacro:novatel_smart6 prefix="$(optenv JACKAL_NAVSAT_MOUNT rear)"/>
     <joint name="$(optenv JACKAL_NAVSAT_MOUNT rear)_navsat_joint" type="fixed">
       <origin xyz="0 0 0" rpy="0 0 0" />
@@ -186,6 +167,4 @@
         prefix="front"
         parent_link="front_fender_accessory_link"
-        min_angle="${-pi/2}"
-        max_angle="${pi/2}"
         topic="$(optenv JACKAL_FRONT_LASER_TOPIC front/scan)">
         <origin xyz="0 0 0" rpy="0 0 0" />
@@ -198,6 +177,4 @@
         prefix="rear"
         parent_link="rear_fender_accessory_link"
-        min_angle="${-pi/2}"
-        max_angle="${pi/2}"
         topic="$(optenv JACKAL_REAR_LASER_TOPIC rear/scan)">
         <origin xyz="0 0 0" rpy="0 0 0" />
