Commit message: Rebase from 'upstream'

File: jackal_description/urdf/accessories/bridge_plate.urdf.xacro (robot description, xacro)
@@ -1,11 +1,17 @@
 <?xml version="1.0"?>
 <robot xmlns:xacro="http://www.ros.org/wiki/xacro">
-  <xacro:macro name="bridge_plate" params="mount height">
-    <joint name="${mount}_mount_to_${mount}_bridge" type="fixed">
-      <parent link="${mount}_mount"/>
-      <child link="${mount}_bridge"/>
+  <xacro:macro name="bridge_plate" params="prefix parent height *origin">
+    <link name="${prefix}_bridge_base"/>
+    <joint name="${prefix}_bridge_base_joint" type="fixed">
+      <parent link="${parent}"/>
+      <child link="${prefix}_bridge_base" />
+      <xacro:insert_block name="origin" />
+    </joint>
+    <joint name="${prefix}_bridge_joint" type="fixed">
+      <parent link="${prefix}_bridge_base"/>
+      <child link="${prefix}_bridge"/>
       <origin xyz="0.0 0.0 ${height}" rpy="0 0 0"/>
     </joint>
-    <link name="${mount}_bridge">
+    <link name="${prefix}_bridge">
       <visual>
         <origin xyz="0 0 0" rpy="1.5707 0.0 1.5707" />
@@ -16,5 +22,5 @@
       </visual>
     </link>
-    <standoff_box mount="${mount}" height="${height}" />
+    <xacro:standoff_box prefix="${prefix}" parent="${prefix}_bridge_base" height="${height}" />
   </xacro:macro>
 </robot>

File: jackal_description/urdf/accessories/novatel_smart7.urdf.xacro (robot description, xacro)
@@ -20,3 +20,25 @@
     </link>
   </xacro:macro>
+  <xacro:macro name="novatel_smart7_stand" params="prefix parent height:=14.5 *origin">
+    <link name="${prefix}_navsat_stand">
+      <visual>
+        <origin xyz="0 0 ${height/2}" rpy="0 0 0"/>
+        <geometry>
+          <box size="0.045 0.025 ${height}" />
+        </geometry>
+        <material name="black" />
+      </visual>
+      <collision>
+        <origin xyz="0 0 ${height/2}" rpy="0 0 0"/>
+        <geometry>
+          <box size="0.045 0.025 ${height}" />
+        </geometry>
+      </collision>
+    </link>
+    <joint name="${prefix}_navsat_stand_joint" type="fixed">
+      <xacro:insert_block name="origin" />
+      <parent link="${parent}" />
+      <child link="${prefix}_navsat_stand" />
+    </joint>
+  </xacro:macro>
 </robot>

File: jackal_description/urdf/accessories/standoffs.urdf.xacro (robot description, xacro)
@@ -19,17 +19,17 @@
   </xacro:macro>
   <!-- Generate a set of four standoffs from a payload mount point. -->
-  <xacro:macro name="standoff_box" params="mount height">
-    <standoff name="${mount}_standoff0" length="${height}" parent="${mount}_mount">
+  <xacro:macro name="standoff_box" params="prefix parent height">
+    <xacro:standoff name="${prefix}_standoff0" length="${height}" parent="${parent}">
       <origin xyz="0.060 0.060 0" rpy="0 0 0"/>
-    </standoff>
-    <standoff name="${mount}_standoff1" length="${height}" parent="${mount}_mount">
+    </xacro:standoff>
+    <xacro:standoff name="${prefix}_standoff1" length="${height}" parent="${parent}">
       <origin xyz="0.060 -0.060 0" rpy="0 0 0"/>
-    </standoff>
-    <standoff name="${mount}_standoff2" length="${height}" parent="${mount}_mount">
+    </xacro:standoff>
+    <xacro:standoff name="${prefix}_standoff2" length="${height}" parent="${parent}">
       <origin xyz="-0.060 0.060 0" rpy="0 0 0"/>
-    </standoff>
-    <standoff name="${mount}_standoff3" length="${height}" parent="${mount}_mount">
+    </xacro:standoff>
+    <xacro:standoff name="${prefix}_standoff3" length="${height}" parent="${parent}">
       <origin xyz="-0.060 -0.060 0" rpy="0 0 0"/>
-    </standoff>
+    </xacro:standoff>
   </xacro:macro>
 </robot>
