Commit message: Imported upstream version '1.0.2' of 'upstream'

File: jackal_description/urdf/accessories.urdf.xacro (robot description, xacro)
@@ -14,28 +14,9 @@
   <xacro:include filename="$(find jackal_description)/urdf/accessories/bridge_plate.urdf.xacro" />
   <!-- 2D Lidars -->
-  <xacro:include filename="$(find sick_tim)/urdf/sick_tim.urdf.xacro" />
-  <xacro:include filename="$(find lms1xx)/urdf/sick_lms1xx.urdf.xacro" />
-  <xacro:include filename="$(find jackal_description)/urdf/accessories/sick_lms1xx_inverted_mount.urdf.xacro" />
-  <xacro:include filename="$(find jackal_description)/urdf/accessories/sick_lms1xx_upright_mount.urdf.xacro" />
-  <xacro:include filename="$(find jackal_description)/urdf/accessories/hokuyo_utm30.urdf.xacro" />
+  <!-- <xacro:include filename="$(find lms1xx)/urdf/sick_lms1xx.urdf.xacro" />
+  <xacro:include filename="$(find jackal_description)/urdf/accessories/sick_lms1xx_mount.urdf.xacro" />-->
   <xacro:include filename="$(find jackal_description)/urdf/accessories/hokuyo_ust10.urdf.xacro" />
   <xacro:include filename="$(find jackal_description)/urdf/accessories/vlp16_mount.urdf.xacro" />
   <xacro:include filename="$(find jackal_description)/urdf/accessories/hdl32_mount.urdf.xacro" />
-  <!--
-    Add Microstrain IMU. By default the Jackal comes equipped with an IMU linked to "imu_link". These extra
-    optional microstrain IMU's will be added to another frame, by default, "microstrain_link".
-  -->
-  <xacro:if value="$(optenv JACKAL_IMU_MICROSTRAIN 0)">
-    <xacro:property name="frame"  value="$(optenv JACKAL_IMU_MICROSTRAIN_LINK microstrain_link)"/>
-    <xacro:property name="parent" value="$(optenv JACKAL_IMU_MICROSTRAIN_PARENT base_link)"/>
-    <xacro:property name="xyz"    value="$(optenv JACKAL_IMU_MICROSTRAIN_OFFSET -0.139 0.096 0.100)"/>
-    <xacro:property name="rpy"    value="$(optenv JACKAL_IMU_MICROSTRAIN_RPY ${PI} 0 -${PI/2})"/>
-    <link name="${frame}" />
-    <joint name="${frame}_joint" type="fixed">
-      <parent link="${parent}" />
-      <child link="${frame}" />
-      <origin xyz="${xyz}" rpy="${rpy}" />
-    </joint>
-  </xacro:if>
   <!--
     Add primary/secondary 2D lidar sensors.  By default these are SICK LMS1xx but can be changed with the
@@ -43,5 +24,4 @@
     - lms1xx (default) :: SICK LMS1xx
     - ust10            :: Hokuyo UST10
-    - utm30            :: Hokuyo UTM30
   -->
   <!-- Primary 2D Lidar -->
@@ -52,20 +32,12 @@
     <xacro:property name="prefix" value="$(optenv JACKAL_LASER_PREFIX ${mount})" />
     <xacro:property name="parent" value="$(optenv JACKAL_LASER_PARENT ${mount}_mount)" />
-    <xacro:property name="lidar_model" value="$(optenv JACKAL_LASER_MODEL lms1xx)" />
-    <xacro:property name="mount_type" value="$(optenv JACKAL_LASER_MOUNT_TYPE upright)" />
+    <xacro:property name="lidar_model" value="$(optenv JACKAL_LASER_MODEL ust10)" />
     <!-- SICK LMS1xx -->
     <xacro:if value="${lidar_model == 'lms1xx'}">
       <!-- Mount Enabled -->
       <xacro:if value="${tower}">
-        <xacro:if value="${mount_type == 'upright'}">
-          <xacro:sick_lms1xx_upright_mount topic="${topic}" prefix="${prefix}" parent_link="${parent}">
-            <origin xyz="$(optenv JACKAL_LASER_OFFSET 0 0 0)" rpy="$(optenv JACKAL_LASER_RPY 0 0 0)" />
-          </xacro:sick_lms1xx_upright_mount>
-        </xacro:if>
-        <xacro:if value="${mount_type == 'inverted'}">
-          <xacro:sick_lms1xx_inverted_mount topic="${topic}" prefix="${prefix}" parent_link="${parent}">
-            <origin xyz="$(optenv JACKAL_LASER_OFFSET 0 0 0)" rpy="$(optenv JACKAL_LASER_RPY 0 0 0)" />
-          </xacro:sick_lms1xx_inverted_mount>
-        </xacro:if>
+        <xacro:sick_lms1xx_mount topic="${topic}" prefix="${prefix}" parent_link="${parent}">
+          <origin xyz="$(optenv JACKAL_LASER_OFFSET 0 0 0)" rpy="$(optenv JACKAL_LASER_RPY 0 0 0)" />
+        </xacro:sick_lms1xx_mount>
       </xacro:if>
       <!-- Mount Disabled -->
@@ -85,14 +57,4 @@
       </xacro:unless>
     </xacro:if>
-    <!-- SICK Tim -->
-    <xacro:if value="${lidar_model == 'tim551'}">
-      <xacro:property name="prefix" value="$(optenv JACKAL_LASER_PREFIX tim551)" />
-      <xacro:sick_tim551 name="${prefix}" ros_topic="${topic}"/>
-      <joint name="${prefix}_mount_link_joint" type="fixed">
-        <origin xyz="$(optenv JACKAL_LASER_OFFSET 0 0 0)" rpy="$(optenv JACKAL_LASER_RPY 0 0 0)"/>
-        <parent link="${parent}"/>
-        <child link="${prefix}_mount_link"/>
-      </joint>
-    </xacro:if>
     <!-- Hokuyo UST10 -->
     <xacro:if value="${lidar_model == 'ust10'}">
@@ -100,10 +62,4 @@
         <origin xyz="$(optenv JACKAL_LASER_OFFSET 0 0 0)" rpy="$(optenv JACKAL_LASER_RPY 0 0 0)" />
       </xacro:hokuyo_ust10_mount>
-    </xacro:if>
-    <!-- Hokuyo UTM30 -->
-    <xacro:if value="${lidar_model == 'utm30'}">
-      <xacro:hokuyo_utm30_mount topic="${topic}" prefix="${prefix}" parent_link="${parent}">
-        <origin xyz="$(optenv JACKAL_LASER_OFFSET 0 0 0)" rpy="$(optenv JACKAL_LASER_RPY 0 0 0)" />
-      </xacro:hokuyo_utm30_mount>
     </xacro:if>
   </xacro:if>
@@ -115,5 +71,5 @@
     <xacro:property name="prefix" value="$(optenv JACKAL_LASER_SECONDARY_PREFIX ${mount})" />
     <xacro:property name="parent" value="$(optenv JACKAL_LASER_SECONDARY_PARENT ${mount}_mount)" />
-    <xacro:property name="lidar_model" value="$(optenv JACKAL_LASER_SECONDARY_MODEL lms1xx)" />
+    <xacro:property name="lidar_model" value="$(optenv JACKAL_LASER_SECONDARY_MODEL ust10)" />
     <!-- SICK LMS1xx -->
     <xacro:if value="${lidar_model == 'lms1xx'}">
@@ -140,14 +96,4 @@
       </xacro:unless>
     </xacro:if>
-    <!-- SICK Tim -->
-    <xacro:if value="${lidar_model == 'tim551'}">
-      <xacro:property name="prefix" value="$(optenv JACKAL_LASER_SECONDARY_PREFIX tim551_2)" />
-      <xacro:sick_tim551 name="${prefix}" ros_topic="${topic}"/>
-      <joint name="${prefix}_mount_link_joint" type="fixed">
-        <origin xyz="$(optenv JACKAL_LASER_SECONDARY_OFFSET 0 0 0)" rpy="$(optenv JACKAL_LASER_SECONDARY_RPY 0 0 3.14159)"/>
-        <parent link="${parent}"/>
-        <child link="${prefix}_mount_link"/>
-      </joint>
-    </xacro:if>
     <!-- Hokuyo UST10 -->
     <xacro:if value="${lidar_model == 'ust10'}">
@@ -155,10 +101,4 @@
         <origin xyz="$(optenv JACKAL_LASER_SECONDARY_OFFSET 0 0 0)" rpy="$(optenv JACKAL_LASER_SECONDARY_RPY 0 0 3.14159)" />
       </xacro:hokuyo_ust10_mount>
-    </xacro:if>
-    <!-- Hokuyo UTM30 -->
-    <xacro:if value="${lidar_model == 'utm30'}">
-      <xacro:hokuyo_utm30_mount topic="${topic}" prefix="${prefix}" parent_link="${parent}">
-        <origin xyz="$(optenv JACKAL_LASER_SECONDARY_OFFSET 0 0 0)" rpy="$(optenv JACKAL_LASER_SECONDARY_RPY 0 0 3.14159)" />
-      </xacro:hokuyo_utm30_mount>
     </xacro:if>
   </xacro:if>
@@ -231,10 +171,10 @@
       <!-- Tower Enabled -->
       <xacro:if value="${tower}">
-        <xacro:bridge_plate prefix="${prefix}" parent="${parent}" height="$(optenv JACKAL_NAVSAT_HEIGHT 0.1)">
-          <origin xyz="$(optenv JACKAL_NAVSAT_OFFSET 0 0 0)" rpy="$(optenv JACKAL_NAVSAT_RPY 0 0 0)"/>
-        </xacro:bridge_plate>
+        <xacro:novatel_smart7_stand prefix="${prefix}" parent="${parent}" height="$(optenv JACKAL_NAVSAT_HEIGHT 0.145)">
+          <origin xyz="$(optenv JACKAL_NAVSAT_OFFSET 0 0 0)" rpy="$(optenv JACKAL_NAVSAT_RPY 0 0 0)" />
+        </xacro:novatel_smart7_stand>
         <joint name="${prefix}_navsat_joint" type="fixed">
-          <origin xyz="0 0 0" rpy="0 0 0" />
-          <parent link="${prefix}_bridge" />
+          <origin xyz="0 0 $(optenv JACKAL_NAVSAT_HEIGHT 0.145)" rpy="0 0 0"/>
+          <parent link="${prefix}_navsat_stand" />
           <child link="${prefix}_navsat" />
         </joint>
@@ -258,5 +198,5 @@
   <!-- Common camera mounts and accessory URDFs. -->
   <xacro:include filename="$(find jackal_description)/urdf/accessories/camera_mount.urdf.xacro" />
-  <xacro:include filename="$(find pointgrey_camera_description)/urdf/pointgrey_flea3.urdf.xacro" />
+  <!--xacro:include filename="$(find pointgrey_camera_description)/urdf/pointgrey_flea3.urdf.xacro" /-->
   <!-- If enabled, generate the flea3 camera payload with a tilt of 30 degrees. -->
   <xacro:if value="$(optenv JACKAL_FLEA3 0)">
@@ -338,5 +278,5 @@
   </xacro:if>
   <!-- If enabled, generate the bumblebee2 camera payload with a tilt of 0 degrees. -->
-  <xacro:include filename="$(find pointgrey_camera_description)/urdf/pointgrey_bumblebee2.urdf.xacro" />
+  <!--xacro:include filename="$(find pointgrey_camera_description)/urdf/pointgrey_bumblebee2.urdf.xacro" /-->
   <!-- If enabled, generate the bumblebee2 camera payload with a tilt of 0 degrees. -->
   <!-- Disabled temporarily due to metapackage issue. -->
@@ -380,18 +320,4 @@
     </xacro:unless>
   </xacro:if>
-  <!-- BlackflyS Camera -->
-  <xacro:include filename="$(find flir_camera_description)/urdf/flir_blackflys.urdf.xacro"/>
-  <xacro:if value="$(optenv JACKAL_BLACKFLY 0)">
-    <xacro:property name="prefix" value="$(optenv JACKAL_BLACKFLY_PREFIX front_camera)"/>
-    <xacro:property name="parent" value="$(optenv JACKAL_BLACKFLY_PARENT front_mount)"/>
-    <xacro:property name="xyz"    value="$(optenv JACKAL_BLACKFLY_OFFSET 0 0 0)"/>
-    <xacro:property name="rpy"    value="$(optenv JACKAL_BLACKFLY_RPY    0 0 0)"/>
-    <xacro:flir_blackflys frame="${prefix}"/>
-    <joint name="${prefix}_mount_joint" type="fixed">
-      <child link="${prefix}"/>
-      <parent link="${parent}"/>
-      <origin xyz="0 0 0" rpy="0 0 0"/>
-    </joint>
-  </xacro:if>
   <!-- Fender Accessories -->
   <xacro:if value="$(optenv JACKAL_FRONT_ACCESSORY_FENDER 0)">
@@ -419,26 +345,4 @@
       </xacro:hokuyo_ust10_mount>
     </xacro:if>
-  </xacro:if>
-  <!-- Bumper Accessories -->
-  <xacro:if value="$(optenv JACKAL_WIBOTIC_BUMPER 0)">
-    <link name="wibotic_bumper">
-      <visual>
-        <geometry>
-          <mesh filename="package://jackal_description/meshes/wibotic_bumper.stl" />
-        </geometry>
-        <material name="dark_grey" />
-      </visual>
-      <collision>
-        <geometry>
-          <box size="0.115 0.25 0.145"/>
-        </geometry>
-        <origin xyz="-0.017575 0 0.0575" rpy="0 0 0"/>
-      </collision>
-    </link>
-    <joint name="wibotic_bumper_joint" type="fixed">
-      <origin xyz="0.285 0 0.07455" rpy="0 0 0"/>
-      <parent link="base_link"/>
-      <child link="wibotic_bumper"/>
-    </joint>
   </xacro:if>
   <xacro:if value="$(optenv JACKAL_ARK_ENCLOSURE 0)">
