Commit message: Imported upstream version '0.8.1' of 'upstream'

File: jackal_description/urdf/accessories/hokuyo_ust10.urdf.xacro (robot description, xacro)
@@ -1,7 +1,7 @@
 <?xml version="1.0"?>
 <robot xmlns:xacro="http://ros.org/wiki/xacro">
-  <xacro:macro name="hokuyo_ust10_mount" params="prefix topic parent_link min_angle:=-2.35619 max_angle:=2.35619 *origin">
+  <xacro:macro name="hokuyo_ust10_mount" params="prefix topic parent_link *origin">
     <xacro:macro name="hokuyo_ust10" params="frame:=laser topic:=scan sample_size:=720 update_rate:=50
-               min_angle:=${min_angle} max_angle:=${max_angle} min_range:=0.1 max_range:=30.0 robot_namespace:=/">
+               min_angle:=-2.35619 max_angle:=2.35619 min_range:=0.1 max_range:=30.0 robot_namespace:=/">
       <link name="${frame}">
         <inertial>

File: jackal_description/urdf/accessories/vlp16_mount.urdf.xacro (robot description, xacro)
@@ -1,99 +1,92 @@
 <robot xmlns:xacro="http://wiki.ros.org/xacro">
   <xacro:include filename="$(find velodyne_description)/urdf/VLP-16.urdf.xacro" />
-  <xacro:macro name="vlp16_mount" params="prefix parent_link topic tower height:=0.1 *origin">
-    <xacro:if value="${tower}">
-      <link name="${prefix}_vlp16_mount" />
-      <link name="${prefix}_vlp16_plate">
-        <visual>
-          <geometry>
-            <box size="0.1 0.1 0.002" />
-          </geometry>
-          <material name="black" />
-          <origin xyz="0 0 -0.001" rpy="0 0 0" />
-        </visual>
-      </link>
-      <link name="${prefix}_vlp16_leg1">
-        <visual>
-          <geometry>
-            <cylinder length="${height}" radius="0.003" />
-          </geometry>
-          <material name="white">
-            <color rgba="1 1 1 1" />
-          </material>
-          <origin xyz="0 0 ${height/2}" rpy="0 0 0" />
-        </visual>
-      </link>
-      <link name="${prefix}_vlp16_leg2">
-        <visual>
-          <geometry>
-            <cylinder length="${height}" radius="0.003" />
-          </geometry>
-          <material name="white">
-            <color rgba="1 1 1 1" />
-          </material>
-          <origin xyz="0 0 ${height/2}" rpy="0 0 0" />
-        </visual>
-      </link>
-      <link name="${prefix}_vlp16_leg3">
-        <visual>
-          <geometry>
-            <cylinder length="${height}" radius="0.003" />
-          </geometry>
-          <material name="white">
-            <color rgba="1 1 1 1" />
-          </material>
-          <origin xyz="0 0 ${height/2}" rpy="0 0 0" />
-        </visual>
-      </link>
-      <link name="${prefix}_vlp16_leg4">
-        <visual>
-          <geometry>
-            <cylinder length="${height}" radius="0.003" />
-          </geometry>
-          <material name="white">
-            <color rgba="1 1 1 1" />
-          </material>
-          <origin xyz="0 0 ${height/2}" rpy="0 0 0" />
-        </visual>
-      </link>
-      <joint name="${prefix}_vlp16_mount_joint" type="fixed">
-        <parent link="${parent_link}" />
-        <child link="${prefix}_vlp16_mount" />
-        <xacro:insert_block name="origin" />
-      </joint>
-      <joint name="${prefix}_vlp16_leg1_joint" type="fixed">
-        <parent link="${prefix}_vlp16_mount" />
-        <child link="${prefix}_vlp16_leg1" />
-        <origin xyz="0.05 0.05 0" rpy="0 0 0" />
-      </joint>
-      <joint name="${prefix}_vlp16_leg2_joint" type="fixed">
-        <parent link="${prefix}_vlp16_mount" />
-        <child link="${prefix}_vlp16_leg2" />
-        <origin xyz="0.05 -0.05 0" rpy="0 0 0" />
-      </joint>
-      <joint name="${prefix}_vlp16_leg3_joint" type="fixed">
-        <parent link="${prefix}_vlp16_mount" />
-        <child link="${prefix}_vlp16_leg3" />
-        <origin xyz="-0.05 0.05 0" rpy="0 0 0" />
-      </joint>
-      <joint name="${prefix}_vlp16_leg4_joint" type="fixed">
-        <parent link="${prefix}_vlp16_mount" />
-        <child link="${prefix}_vlp16_leg4" />
-        <origin xyz="-0.05 -0.05 0" rpy="0 0 0" />
-      </joint>
-      <joint name="${prefix}_vlp16_plate_joint" type="fixed">
-        <parent link="${prefix}_vlp16_mount" />
-        <child link="${prefix}_vlp16_plate" />
-        <origin xyz="0 0 ${height}" rpy="0 0 0" />
-      </joint>
-      <xacro:VLP-16 parent="${prefix}_vlp16_plate" topic="${topic}">
-        <origin xyz="0 0 0" rpy="0 0 0" />
-      </xacro:VLP-16>
-    </xacro:if>
-    <xacro:unless value="${tower}">
-      <xacro:VLP-16 parent="${parent_link}" topic="${topic}">
-        <xacro:insert_block name="origin" />
-      </xacro:VLP-16>
-    </xacro:unless>
+  <xacro:macro name="vlp16_mount" params="prefix parent_link topic height:=0.1 *origin">
+    <link name="${prefix}_vlp16_mount" />
+    <link name="${prefix}_vlp16_plate">
+      <visual>
+        <geometry>
+          <box size="0.1 0.1 0.002" />
+        </geometry>
+        <material name="black" />
+        <origin xyz="0 0 -0.001" rpy="0 0 0" />
+      </visual>
+    </link>
+    <link name="${prefix}_vlp16_leg1">
+      <visual>
+        <geometry>
+          <cylinder length="${height}" radius="0.003" />
+        </geometry>
+        <material name="white">
+          <color rgba="1 1 1 1" />
+        </material>
+        <origin xyz="0 0 ${height/2}" rpy="0 0 0" />
+      </visual>
+    </link>
+    <link name="${prefix}_vlp16_leg2">
+      <visual>
+        <geometry>
+          <cylinder length="${height}" radius="0.003" />
+        </geometry>
+        <material name="white">
+          <color rgba="1 1 1 1" />
+        </material>
+        <origin xyz="0 0 ${height/2}" rpy="0 0 0" />
+      </visual>
+    </link>
+    <link name="${prefix}_vlp16_leg3">
+      <visual>
+        <geometry>
+          <cylinder length="${height}" radius="0.003" />
+        </geometry>
+        <material name="white">
+          <color rgba="1 1 1 1" />
+        </material>
+        <origin xyz="0 0 ${height/2}" rpy="0 0 0" />
+      </visual>
+    </link>
+    <link name="${prefix}_vlp16_leg4">
+      <visual>
+        <geometry>
+          <cylinder length="${height}" radius="0.003" />
+        </geometry>
+        <material name="white">
+          <color rgba="1 1 1 1" />
+        </material>
+        <origin xyz="0 0 ${height/2}" rpy="0 0 0" />
+      </visual>
+    </link>
+    <joint name="${prefix}_vlp16_mount_joint" type="fixed">
+      <parent link="${parent_link}" />
+      <child link="${prefix}_vlp16_mount" />
+      <xacro:insert_block name="origin" />
+    </joint>
+    <joint name="${prefix}_vlp16_leg1_joint" type="fixed">
+      <parent link="${prefix}_mount" />
+      <child link="${prefix}_vlp16_leg1" />
+      <origin xyz="0.05 0.05 0" rpy="0 0 0" />
+    </joint>
+    <joint name="${prefix}_vlp16_leg2_joint" type="fixed">
+      <parent link="${prefix}_mount" />
+      <child link="${prefix}_vlp16_leg2" />
+      <origin xyz="0.05 -0.05 0" rpy="0 0 0" />
+    </joint>
+    <joint name="${prefix}_vlp16_leg3_joint" type="fixed">
+      <parent link="${prefix}_mount" />
+      <child link="${prefix}_vlp16_leg3" />
+      <origin xyz="-0.05 0.05 0" rpy="0 0 0" />
+    </joint>
+    <joint name="${prefix}_vlp16_leg4_joint" type="fixed">
+      <parent link="${prefix}_mount" />
+      <child link="${prefix}_vlp16_leg4" />
+      <origin xyz="-0.05 -0.05 0" rpy="0 0 0" />
+    </joint>
+    <joint name="${prefix}_vlp16_plate_joint" type="fixed">
+      <parent link="${prefix}_vlp16_mount" />
+      <child link="${prefix}_vlp16_plate" />
+      <origin xyz="0 0 ${height}" rpy="0 0 0" />
+    </joint>
+    <xacro:VLP-16 parent="${prefix}_vlp16_plate" topic="${topic}">
+      <origin xyz="0 0 0" rpy="0 0 0" />
+    </xacro:VLP-16>
   </xacro:macro>
 </robot>

File: jackal_description/urdf/jackal.urdf.xacro (robot description, xacro)
@@ -203,16 +203,4 @@
     <origin xyz="-0.180 0.126 0.1815" />
   </joint>
-  <!--
-    Optionally add a GX5 IMU
-  -->
-  <xacro:if value="$(optenv JACKAL_GX5_IMU 0)">
-    <link name="gx5_link" />
-    <joint name="gx5_joint" type="fixed">
-      <parent link="base_link" />
-      <child link="gx5_link" />
-      <!-- TODO This offset & rotation may not be final, but it's good enough for now.  May update, pending RSCI-10 -->
-      <origin xyz="$(optenv JACKAL_GX5_IMU_OFFSET -0.139 0.096 0.100)" rpy="$(optenv JACKAL_GX5_IMU_RPY ${PI} 0 -${PI/2})" />
-    </joint>
-  </xacro:if>
   <link name="mid_mount"></link>
   <joint name="mid_mount_joint" type="fixed">
@@ -241,5 +229,3 @@
   <!-- Optional custom includes. -->
   <xacro:include filename="$(optenv JACKAL_URDF_EXTRAS empty.urdf)" />
-  <!-- Optional for Clearpath internal softwares -->
-  <xacro:include filename="$(optenv CPR_URDF_EXTRAS empty.urdf)" />
 </robot>

Commit message: Imported upstream version '0.8.7' of 'upstream'

File: jackal_description/urdf/accessories/hokuyo_ust10.urdf.xacro (robot description, xacro)
@@ -1,5 +1,5 @@
 <?xml version="1.0"?>
 <robot xmlns:xacro="http://ros.org/wiki/xacro">
-  <xacro:macro name="hokuyo_ust10_mount" params="prefix topic parent_link *origin">
+  <xacro:macro name="hokuyo_ust10_mount" params="prefix topic parent_link min_angle:=-2.35619 max_angle:=2.35619 *origin">
     <xacro:macro name="hokuyo_ust10" params="frame:=laser topic:=scan sample_size:=720 update_rate:=50
                min_angle:=-2.35619 max_angle:=2.35619 min_range:=0.1 max_range:=30.0 robot_namespace:=/">
@@ -39,10 +39,8 @@
             </noise>
           </ray>
-          <plugin name="gazebo_ros_laser" filename="libgazebo_ros_ray_sensor.so">
-            <ros>
-              <namespace>${robot_namespace}</namespace>
-              <remapping>~/out:=${topic}</remapping>
-            </ros>
-            <frame_name>${frame}</frame_name>
+          <plugin name="gazebo_ros_laser" filename="libgazebo_ros_laser.so">
+            <topicName>${topic}</topicName>
+            <frameName>${frame}</frameName>
+            <robotNamespace>${robot_namespace}</robotNamespace>
           </plugin>
         </sensor>

Commit message: Imported upstream version '0.8.7' of 'upstream'

File: jackal_description/urdf/accessories/hokuyo_ust10.urdf.xacro (robot description, xacro)
@@ -1,5 +1,5 @@
 <?xml version="1.0"?>
 <robot xmlns:xacro="http://ros.org/wiki/xacro">
-  <xacro:macro name="hokuyo_ust10_mount" params="prefix topic parent_link *origin">
+  <xacro:macro name="hokuyo_ust10_mount" params="prefix topic parent_link min_angle:=-2.35619 max_angle:=2.35619 *origin">
     <xacro:macro name="hokuyo_ust10" params="frame:=laser topic:=scan sample_size:=720 update_rate:=50
                min_angle:=-2.35619 max_angle:=2.35619 min_range:=0.1 max_range:=30.0 robot_namespace:=/">
@@ -39,11 +39,8 @@
             </noise>
           </ray>
-          <plugin name="gazebo_ros_laser" filename="libgazebo_ros_ray_sensor.so">
-            <ros>
-              <namespace>${robot_namespace}</namespace>
-              <remapping>~/out:=${topic}</remapping>
-            </ros>
-            <output_type>sensor_msgs/LaserScan</output_type>
-            <frame_name>${frame}</frame_name>
+          <plugin name="gazebo_ros_laser" filename="libgazebo_ros_laser.so">
+            <topicName>${topic}</topicName>
+            <frameName>${frame}</frameName>
+            <robotNamespace>${robot_namespace}</robotNamespace>
           </plugin>
         </sensor>
